Commit message: add arm control

File: urdf/aibot_arm.urdf.xacro (robot description, xacro)
@@ -1,5 +1,4 @@
 <?xml version='1.0'?>
-<robot name="bricklayer" xmlns:xacro="http://ros.org/wiki/xacro">
-  <!-- Bricklayer chassis -->
+<robot name="aibot" xmlns:xacro="http://ros.org/wiki/xacro">
   <xacro:include filename="$(find aibot_description)/urdf/arm/arm.urdf.xacro" />
   <xacro:property name="PI" value="3.1415926535897931" />
@@ -10,9 +9,4 @@
   </aibot_arm>
   <!-- gazebo controller plugin -->
-  <!-- <xacro:include filename="$(find bricklayer_description)/controller/ros_controller.urdf.xacro" /> -->
-  <!-- RGBD Camera -->
-  <!-- <xacro:rgbd_camera name="rgbd_camera" parent="chassis">
-    <origin xyz="0.5 0 0.5" rpy="0 0 0"/>
-    <origin xyz="0 0 0" rpy="${-90.0 * deg_to_rad} 0 ${-90.0 * deg_to_rad}"/>
-  </xacro:rgbd_camera> -->
+  <xacro:include filename="$(find aibot_description)/controller/ros_controller.urdf.xacro" />
 </robot>

File: urdf/arm/arm.gazebo.xacro (robot description, xacro)
@@ -8,26 +8,54 @@
       <mu2>0.9</mu2>
     </gazebo>
-    <gazebo reference = "arm_vert_link">
+    <gazebo reference = "arm_base_link_joint">
+      <implicitSpringDamper>true</implicitSpringDamper>
+    </gazebo>
+    <gazebo reference = "arm_base_rot_link">
       <mu1>0.9</mu1>
       <mu2>0.9</mu2>
     </gazebo>
-    <gazebo reference = "arm_hori_link">
+    <gazebo reference = "arm_base_rot_link_joint">
+      <implicitSpringDamper>true</implicitSpringDamper>
+    </gazebo>
+    <gazebo reference = "arm_first_link">
       <mu1>0.9</mu1>
       <mu2>0.9</mu2>
     </gazebo>
-    <gazebo reference = "gripper_rot_link">
+    <gazebo reference = "arm_first_link_joint">
+      <implicitSpringDamper>true</implicitSpringDamper>
+    </gazebo>
+    <gazebo reference = "arm_second_motor_link">
       <mu1>0.9</mu1>
       <mu2>0.9</mu2>
     </gazebo>
-    <gazebo reference = "arm_base_link_joint">
+    <gazebo reference = "arm_second_motor_link_joint">
       <implicitSpringDamper>true</implicitSpringDamper>
     </gazebo>
-    <gazebo reference = "arm_vert_link_joint">
+    <gazebo reference = "arm_second_connector_link">
+      <mu1>0.9</mu1>
+      <mu2>0.9</mu2>
+    </gazebo>
+    <gazebo reference = "arm_second_connector_link_joint">
       <implicitSpringDamper>true</implicitSpringDamper>
     </gazebo>
-    <gazebo reference = "arm_hori_link_joint">
+    <gazebo reference = "arm_second_link">
+      <mu1>0.9</mu1>
+      <mu2>0.9</mu2>
+    </gazebo>
+    <gazebo reference = "arm_second_link_joint">
       <implicitSpringDamper>true</implicitSpringDamper>
     </gazebo>
-    <gazebo reference = "gripper_rot_link_joint">
+    <gazebo reference = "arm_third_link">
+      <mu1>0.9</mu1>
+      <mu2>0.9</mu2>
+    </gazebo>
+    <gazebo reference = "arm_third_link_joint">
+      <implicitSpringDamper>true</implicitSpringDamper>
+    </gazebo>
+    <gazebo reference = "arm_fourth_link">
+      <mu1>0.9</mu1>
+      <mu2>0.9</mu2>
+    </gazebo>
+    <gazebo reference = "arm_fourth_link_joint">
       <implicitSpringDamper>true</implicitSpringDamper>
     </gazebo>

File: urdf/arm/arm.urdf.xacro (robot description, xacro)
@@ -2,7 +2,6 @@
 <robot xmlns:xacro="http://ros.org/wiki/xacro">
   <xacro:include filename ="$(find aibot_description)/urdf/arm/arm.transmission.xacro"/>
-  <xacro:include filename ="$(find aibot_description)/urdf/arm/arm.gazebo.xacro"/>
-  <!-- <xacro:include filename ="$(find aibot_description)/urdf/inertia.xacro"/> -->
-  <!-- <xacro:include filename="$(find aibot_description)/urdf/gripper/gripper.urdf.xacro" /> -->
+  <!-- <xacro:include filename ="$(find aibot_description)/urdf/arm/arm.gazebo.xacro"/> -->
+  <xacro:include filename ="$(find aibot_description)/urdf/arm/inertia.xacro"/>
   <xacro:macro name="aibot_arm" params="parent_link *origin">
     <link name='arm_base_link'>
@@ -22,9 +21,9 @@
       </collision>
       <!-- the physics for gazebo -->
-      <!-- <inertial>
-        <mass value="8.0"/>
+      <inertial>
+        <mass value="200.0"/>
         <origin xyz="0 0 0.96" rpy=" 0 0 0"/>
         <box_inertia m="8.0" x="0.24" y="0.23" z="1.92"/>
-      </inertial>  -->
+      </inertial>
     </link>
     <joint type="fixed" name="arm_base_link_joint">
@@ -46,11 +45,11 @@
         </geometry>
       </collision>
-      <!-- <inertial>
+      <inertial>
         <mass value="8.0"/>
         <origin xyz="0 0 0.96" rpy=" 0 0 0"/>
         <box_inertia m="8.0" x="0.24" y="0.23" z="1.92"/>
-      </inertial>  -->
-    </link>
-    <joint type="revolute" name="arm_base_link_rot_joint">
+      </inertial>
+    </link>
+    <joint type="revolute" name="arm_base_rot_link_joint">
       <origin xyz="0 0 0.0355" rpy="0 0 ${-PI}"/>
       <child link="arm_base_rot_link"/>
@@ -66,17 +65,15 @@
         </geometry>
       </visual>
-      <!-- The Collision of the model -->
-      <collision name='collision'>
-        <origin xyz="0.09331 0 -0.037679" rpy=" 0 0 0"/>
-        <geometry>
-          <box size="2.089 0.296 0.130"/>
-        </geometry>
-      </collision>
-      <!-- the physics for gazebo -->
-      <!-- <inertial>
-        <mass value="6.0"/>
-        <origin xyz="0.09331 0 -0.037679" rpy=" 0 0 0"/>
-        <box_inertia m="6.0" x="2.089" y="0.296" z="0.130"/>
-      </inertial>  -->
+      <collision name='collision'>
+        <origin xyz="0 0 0.96" rpy=" 0 0 0"/>
+        <geometry>
+          <box size="0.24 0.23 1.92"/>
+        </geometry>
+      </collision>
+      <inertial>
+        <mass value="8.0"/>
+        <origin xyz="0 0 0.96" rpy=" 0 0 0"/>
+        <box_inertia m="8.0" x="0.24" y="0.23" z="1.92"/>
+      </inertial>
     </link>
     <joint type="revolute" name="arm_first_link_joint">
@@ -85,5 +82,5 @@
       <parent link="arm_base_rot_link"/>
       <axis xyz="0 1 0" />
-      <limit effort="100000.0" lower="0" upper="1.47" velocity="0.0833"/>
+      <limit effort="100000.0" lower="0" upper="1.47" velocity="0"/>
     </joint>
     <link name = "arm_second_motor_link">
@@ -94,18 +91,16 @@
         </geometry>
       </visual>
-      <!-- The Collision of the model -->
-      <collision name='collision'>
-        <origin xyz="0.09331 0 -0.037679" rpy=" 0 0 0"/>
-        <geometry>
-          <box size="2.089 0.296 0.130"/>
-        </geometry>
-      </collision>
-      <!-- the physics for gazebo -->
-      <!-- <inertial>
-        <mass value="6.0"/>
-        <origin xyz="0.09331 0 -0.037679" rpy=" 0 0 0"/>
-        <box_inertia m="6.0" x="2.089" y="0.296" z="0.130"/>
-      </inertial>  -->
-    </link>arm_second_connector_link
+      <collision name='collision'>
+        <origin xyz="0.09331 0 -0.037679" rpy=" 0 0 0"/>
+        <geometry>
+          <box size="2.089 0.296 0.130"/>
+        </geometry>
+      </collision>
+      <inertial>
+        <mass value="6.0"/>
+        <origin xyz="0.09331 0 -0.037679" rpy=" 0 0 0"/>
+        <box_inertia m="6.0" x="2.089" y="0.296" z="0.130"/>
+      </inertial>
+    </link>
     <joint type="revolute" name="arm_second_motor_link_joint">
       <origin xyz="0 0.0245 0" rpy="0 0 0"/>
@@ -122,17 +117,15 @@
         </geometry>
       </visual>
-      <!-- The Collision of the model -->
-      <collision name='collision'>
-        <origin xyz="0.09331 0 -0.037679" rpy=" 0 0 0"/>
-        <geometry>
-          <box size="2.089 0.296 0.130"/>
-        </geometry>
-      </collision>
-      <!-- the physics for gazebo -->
-      <!-- <inertial>
-        <mass value="6.0"/>
-        <origin xyz="0.09331 0 -0.037679" rpy=" 0 0 0"/>
-        <box_inertia m="6.0" x="2.089" y="0.296" z="0.130"/>
-      </inertial>  -->
+      <collision name='collision'>
+        <origin xyz="0.09331 0 -0.037679" rpy=" 0 0 0"/>
+        <geometry>
+          <box size="2.089 0.296 0.130"/>
+        </geometry>
+      </collision>
+      <inertial>
+        <mass value="6.0"/>
+        <origin xyz="0.09331 0 -0.037679" rpy=" 0 0 0"/>
+        <box_inertia m="6.0" x="2.089" y="0.296" z="0.130"/>
+      </inertial>
     </link>
     <joint type="revolute" name="arm_second_connector_link_joint">
@@ -150,17 +143,15 @@
         </geometry>
       </visual>
-      <!-- The Collision of the model -->
-      <collision name='collision'>
-        <origin xyz="0.09331 0 -0.037679" rpy=" 0 0 0"/>
-        <geometry>
-          <box size="2.089 0.296 0.130"/>
-        </geometry>
-      </collision>
-      <!-- the physics for gazebo -->
-      <!-- <inertial>
-        <mass value="6.0"/>
-        <origin xyz="0.09331 0 -0.037679" rpy=" 0 0 0"/>
-        <box_inertia m="6.0" x="2.089" y="0.296" z="0.130"/>
-      </inertial>  -->
+      <collision name='collision'>
+        <origin xyz="0.09331 0 -0.037679" rpy=" 0 0 0"/>
+        <geometry>
+          <box size="2.089 0.296 0.130"/>
+        </geometry>
+      </collision>
+      <inertial>
+        <mass value="6.0"/>
+        <origin xyz="0.09331 0 -0.037679" rpy=" 0 0 0"/>
+        <box_inertia m="6.0" x="2.089" y="0.296" z="0.130"/>
+      </inertial>
     </link>
     <joint type="revolute" name="arm_second_link_joint">
@@ -178,17 +169,15 @@
         </geometry>
       </visual>
-      <!-- The Collision of the model -->
-      <collision name='collision'>
-        <origin xyz="0.09331 0 -0.037679" rpy=" 0 0 0"/>
-        <geometry>
-          <box size="2.089 0.296 0.130"/>
-        </geometry>
-      </collision>
-      <!-- the physics for gazebo -->
-      <!-- <inertial>
-        <mass value="6.0"/>
-        <origin xyz="0.09331 0 -0.037679" rpy=" 0 0 0"/>
-        <box_inertia m="6.0" x="2.089" y="0.296" z="0.130"/>
-      </inertial>  -->
+      <collision name='collision'>
+        <origin xyz="0.09331 0 -0.037679" rpy=" 0 0 0"/>
+        <geometry>
+          <box size="2.089 0.296 0.130"/>
+        </geometry>
+      </collision>
+      <inertial>
+        <mass value="6.0"/>
+        <origin xyz="0.09331 0 -0.037679" rpy=" 0 0 0"/>
+        <box_inertia m="6.0" x="2.089" y="0.296" z="0.130"/>
+      </inertial>
     </link>
     <joint type="revolute" name="arm_third_link_joint">
@@ -206,17 +195,15 @@
         </geometry>
       </visual>
-      <!-- The Collision of the model -->
-      <collision name='collision'>
-        <origin xyz="0.09331 0 -0.037679" rpy=" 0 0 0"/>
-        <geometry>
-          <box size="2.089 0.296 0.130"/>
-        </geometry>
-      </collision>
-      <!-- the physics for gazebo -->
-      <!-- <inertial>
-        <mass value="6.0"/>
-        <origin xyz="0.09331 0 -0.037679" rpy=" 0 0 0"/>
-        <box_inertia m="6.0" x="2.089" y="0.296" z="0.130"/>
-      </inertial>  -->
+      <collision name='collision'>
+        <origin xyz="0.09331 0 -0.037679" rpy=" 0 0 0"/>
+        <geometry>
+          <box size="2.089 0.296 0.130"/>
+        </geometry>
+      </collision>
+      <inertial>
+        <mass value="6.0"/>
+        <origin xyz="0.09331 0 -0.037679" rpy=" 0 0 0"/>
+        <box_inertia m="6.0" x="2.089" y="0.296" z="0.130"/>
+      </inertial>
     </link>
     <joint type="revolute" name="arm_fourth_link_joint">
@@ -227,4 +214,13 @@
       <limit effort="100000.0" lower="-${PI}" upper="1.47" velocity="0.0833"/>
     </joint>
+    <!-- <arm_simple_transmission name = "arm_base_link"             reduction = "1.0"/> -->
+    <!-- <arm_simple_transmission name = "arm_base_rot_link"         reduction = "1.0"/>
+    <arm_simple_transmission name = "arm_first_link"            reduction = "1.0"/>
+    <arm_simple_transmission name = "arm_second_motor_link"     reduction = "1.0"/>
+    <arm_simple_transmission name = "arm_second_connector_link" reduction = "1.0"/>
+    <arm_simple_transmission name = "arm_second_link"           reduction = "1.0"/>
+    <arm_simple_transmission name = "arm_fourth_link"           reduction = "1.0"/> -->
+    <!-- <arm_gazebo>
+    </arm_gazebo> -->
   </xacro:macro>
 </robot>

Commit message: reform code

File: urdf/aibot_arm.urdf.xacro (robot description, xacro)
@@ -9,4 +9,4 @@
   </aibot_arm>
   <!-- gazebo controller plugin -->
-  <xacro:include filename="$(find aibot_description)/controller/ros_controller.urdf.xacro" />
+  <xacro:include filename="$(find aibot_description)/urdf/controller/ros_controller.urdf.xacro" />
 </robot>

File: urdf/arm/arm.urdf.xacro (robot description, xacro)
@@ -56,5 +56,5 @@
       <parent link="arm_base_link"/>
       <axis xyz="0 0 1" />
-      <limit effort="100.0" lower="0" upper="${2 * PI - 0.01}" velocity="0.3539"/>
+      <limit effort="100.0" lower="0" upper="${2 * PI - 0.01}" velocity="0.70"/>
     </joint>
      <link name = "arm_first_link">
@@ -108,5 +108,5 @@
       <parent link="arm_first_link"/>
       <axis xyz="0 1 0" />
-      <limit effort="100000.0" lower="0" upper="1.47" velocity="0.0833"/>
+      <limit effort="100000.0" lower="0" upper="1.47" velocity="0.833"/>
     </joint>
     <link name = "arm_second_connector_link">
@@ -134,5 +134,5 @@
       <parent link="arm_second_motor_link"/>
       <axis xyz="0 1 0" />
-      <limit effort="100000.0" lower="-${PI}" upper="1.47" velocity="0.0833"/>
+      <limit effort="100000.0" lower="-${PI}" upper="1.47" velocity="0.833"/>
     </joint>
     <link name = "arm_second_link">
@@ -160,5 +160,5 @@
       <parent link="arm_first_link"/>
       <axis xyz="0 1 0" />
-      <limit effort="100000.0" lower="-${PI}" upper="1.47" velocity="0.0833"/>
+      <limit effort="100000.0" lower="-${PI}" upper="1.47" velocity="0.833"/>
     </joint>
     <link name = "arm_third_link">
@@ -186,5 +186,5 @@
       <parent link="arm_second_link"/>
       <axis xyz="0 0 1" />
-      <limit effort="100000.0" lower="-${PI}" upper="1.47" velocity="0.0833"/>
+      <limit effort="100000.0" lower="-${PI}" upper="1.47" velocity="0.833"/>
     </joint>
     <link name = "arm_fourth_link">
@@ -212,13 +212,13 @@
       <parent link="arm_third_link"/>
       <axis xyz="0 1 0" />
-      <limit effort="100000.0" lower="-${PI}" upper="1.47" velocity="0.0833"/>
-    </joint>
-    <!-- <arm_simple_transmission name = "arm_base_link"             reduction = "1.0"/> -->
-    <!-- <arm_simple_transmission name = "arm_base_rot_link"         reduction = "1.0"/>
+      <limit effort="100000.0" lower="-${PI}" upper="1.47" velocity="0.833"/>
+    </joint>
+    <arm_simple_transmission name = "arm_base_link"             reduction = "1.0"/>
+    <arm_simple_transmission name = "arm_base_rot_link"         reduction = "1.0"/>
     <arm_simple_transmission name = "arm_first_link"            reduction = "1.0"/>
     <arm_simple_transmission name = "arm_second_motor_link"     reduction = "1.0"/>
     <arm_simple_transmission name = "arm_second_connector_link" reduction = "1.0"/>
-    <arm_simple_transmission name = "arm_second_link"           reduction = "1.0"/>
-    <arm_simple_transmission name = "arm_fourth_link"           reduction = "1.0"/> -->
+    <arm_simple_transmission name = "arm_third_link"            reduction = "1.0"/>
+    <arm_simple_transmission name = "arm_fourth_link"           reduction = "1.0"/>
     <!-- <arm_gazebo>
     </arm_gazebo> -->
