Commit message: add pump_support

File: urdf/aibot_car.urdf.xacro (robot description, xacro)
@@ -130,5 +130,5 @@
         <cylinder radius="0.005" length="0.005"/>
       </geometry>
-      <material name="green"/>
+      <material name="black"/>
     </visual>
   </link>
@@ -150,5 +150,5 @@
         <cylinder radius="0.03" length="0.017"/>
       </geometry>
-      <material name="green"/>
+      <material name="green_black"/>
     </visual>
   </link>
@@ -181,4 +181,26 @@
     <child link="arm_base_connect"/>
   </joint>
+  <link name="pump_support_link">
+    <collision name='collision_pump_support'>
+     <origin xyz="0 0 0" rpy="0 0 0"/>
+      <geometry>
+        <mesh filename="package://aibot_description/meshes/pump_support.stl" scale="0.001 0.001 0.001"/>
+      </geometry>
+    </collision>
+    <visual>
+      <origin xyz="0 0 0" rpy="1.57 0 1.57"/>
+      <geometry>
+        <mesh filename="package://aibot_description/meshes/pump_support.stl" scale="0.001 0.001 0.001"/>
+      </geometry>
+      <material name = "green_gray">
+        <color rgba = "0.2 0.8 0.6 1"/>
+      </material>
+    </visual>
+  </link>
+  <joint name="pump_support_joint" type="fixed">
+    <origin xyz="0 -0.049 0.02" rpy="0 0 0"/>
+    <parent link="arm_base_connect"/>
+    <child link="pump_support_link"/>
+  </joint>
   <link name="camera_support_link">
     <collision name='collision_camera_support'>
@@ -193,5 +215,5 @@
       </geometry>
       <origin xyz = "0 0 0" rpy = "0 1.57 3.14"/>
-      <material name = "blue">
+      <material name = "green">
         <color rgba = "0 1 0 1"/>
       </material>
@@ -389,7 +411,8 @@
     <visual>
       <geometry>
-        <cylinder length="0.08" radius="0.0125"/>
-      </geometry>
-      <origin xyz = "0.0 0 0 " rpy = "0 0 0"/>
+        <!-- <cylinder length="0.08" radius="0.0125"/> -->
+        <mesh filename="package://aibot_description/meshes/sucker.stl"  scale="0.001 0.001 0.001"/>
+      </geometry>
+      <origin xyz = "0.0 0 0 " rpy = "-1.57 0 1.57"/>
       <material name = "white">
         <color rgba = "0.9 0.9 0.9 1"/>
@@ -398,5 +421,5 @@
     <collision>
       <geometry>
-        <cylinder length="0.08" radius="0.0125"/>
+        <cylinder length="0.06" radius="0.0125"/>
       </geometry>
       <origin xyz = "0.0 0 0 " rpy = "0 0 0"/>
@@ -406,5 +429,6 @@
     <parent link="joint6_flange"/>
     <child link="sucker_joint"/>
-    <origin xyz= "0 0.027 0.0125" rpy = "0 0 0"/>
+    <!-- <origin xyz= "0 0.027 0.0125" rpy = "0 0 0"/> -->
+    <origin xyz= "0 0.022 0" rpy = "0 0 0"/>
   </joint>
 </robot>

Commit message: fix tf name

File: urdf/aibot_car.urdf.xacro (robot description, xacro)
@@ -5,5 +5,5 @@
   <xacro:property name="width" value=".2" />
   <link name='base_link' />
-  <link name='chassis'>
+  <link name='base_footprint'>
     <collision name='collision_body'>
     <origin xyz="0 0 0.045" rpy="0 0 0"/>
@@ -18,5 +18,5 @@
       </geometry>
     </collision>
-    <visual name='chassis_visual'>
+    <visual name='base_footprint_visual'>
       <origin xyz="0 0 0" rpy="1.57 0 0"/>
       <geometry>
@@ -25,7 +25,7 @@
     </visual>
   </link>
-  <joint type="fixed" name="base_chassis">
+  <joint type="fixed" name="base_footprint_joint">
     <origin xyz="0 0 0.016" rpy="0 0 0"/>
-    <child link="chassis"/>
+    <child link="base_footprint"/>
     <parent link="base_link"/>
   </joint>
@@ -61,5 +61,5 @@
     <origin xyz="0.1035 0.09 0.019" rpy="0 0 0"/>
     <child link="front_left_wheel"/>
-    <parent link="chassis"/>
+    <parent link="base_footprint"/>
     <axis xyz="0 1 0" rpy="0 0 0"/>
     <limit effort="10000" velocity="1000"/>
@@ -69,5 +69,5 @@
     <origin xyz="0.1035 -0.09 0.019" rpy="0 0 0"/>
     <child link="front_right_wheel"/>
-    <parent link="chassis"/>
+    <parent link="base_footprint"/>
     <axis xyz="0 1 0" rpy="0 0 0"/>
     <limit effort="10000" velocity="1000"/>
@@ -105,5 +105,5 @@
     <origin xyz="-0.1035 0.09 0.019" rpy="0 0 0"/>
     <child link="rear_left_wheel"/>
-    <parent link="chassis"/>
+    <parent link="base_footprint"/>
     <axis xyz="0 1 0" rpy="0 0 0"/>
     <limit effort="10000" velocity="1000"/>
@@ -113,5 +113,5 @@
     <origin xyz="-0.1035 -0.09 0.019" rpy="0 0 0"/>
     <child link="rear_right_wheel"/>
-    <parent link="chassis"/>
+    <parent link="base_footprint"/>
     <axis xyz="0 1 0" rpy="0 0 0"/>
     <limit effort="10000" velocity="1000"/>
@@ -135,8 +135,8 @@
   <joint name="camera_joint" type="fixed">
     <origin xyz=".12 0 0.0732" rpy="1.57 0 1.57"/>
-    <parent link="chassis"/>
+    <parent link="base_footprint"/>
     <child link="camera"/>
   </joint>
-  <link name="lidar">
+  <link name="laser">
     <collision>
       <origin xyz="0 0 0" rpy="0 0 0"/>
@@ -155,7 +155,7 @@
   <joint name="lidar_joint" type="fixed">
     <axis xyz="0 1 0" />
-    <origin xyz=".0493 0 0.115" rpy="0 0 0"/>
-    <parent link="chassis"/>
-    <child link="lidar"/>
+    <origin xyz=".0493 0 0.115" rpy="0 0 3.14"/>
+    <parent link="base_footprint"/>
+    <child link="laser"/>
   </joint>
   <link name="arm_base_connect">
@@ -178,5 +178,5 @@
   <joint name="arm_base_connect_joint" type="fixed">
     <origin xyz="-0.0865 0 0.0915" rpy="0 0 0"/>
-    <parent link="chassis"/>
+    <parent link="base_footprint"/>
     <child link="arm_base_connect"/>
   </joint>

Commit message: clean code

File: urdf/aibot_car.urdf.xacro (robot description, xacro)
@@ -1,13 +1,16 @@
 <?xml version='1.0'?>
 <robot name="aibot" xmlns:xacro="http://ros.org/wiki/xacro">
-  <xacro:property name="cameraSize" value="0.02"/>
-  <xacro:property name="cameraMass" value="0.1"/>
-  <xacro:property name="width" value=".2" />
   <link name='base_link' />
   <link name='base_footprint'>
+    <visual name='base_footprint_visual'>
+      <origin xyz="0 0 0" rpy="1.57 0 0"/>
+      <geometry>
+        <mesh filename="package://aibot_description/meshes/car_body.stl" scale="0.001 0.001 0.001"/>
+      </geometry>
+    </visual>
     <collision name='collision_body'>
     <origin xyz="0 0 0.045" rpy="0 0 0"/>
       <geometry>
-        <box size=".32 .18 .09"/>
+        <box size="0.32 0.18 0.09"/>
       </geometry>
     </collision>
@@ -15,15 +18,9 @@
      <origin xyz="0.045 0 0.055" rpy="0 0 0"/>
       <geometry>
-        <box size=".12 .1 .11"/>
-      </geometry>
-    </collision>
-    <visual name='base_footprint_visual'>
-      <origin xyz="0 0 0" rpy="1.57 0 0"/>
-      <geometry>
-        <mesh filename="package://aibot_description/meshes/car_body.stl" scale="0.001 0.001 0.001"/>
-      </geometry>
-    </visual>
-  </link>
-  <joint type="fixed" name="base_footprint_joint">
+        <box size="0.12 0.1 0.11"/>
+      </geometry>
+    </collision>
+  </link>
+  <joint name="base_footprint_joint" type="fixed" >
     <origin xyz="0 0 0.016" rpy="0 0 0"/>
     <child link="base_footprint"/>
@@ -31,25 +28,19 @@
   </joint>
   <link name="front_left_wheel">
-    <collision name="collision">
-      <origin xyz="0 0 0" rpy="0 1.5707 1.5707"/>
-      <geometry>
-        <cylinder radius="0.0325" length="0.03"/>
-      </geometry>
-    </collision>
-    <visual name="left_wheel_visual">
-      <origin xyz="0 0 0" rpy="0 1.5707 1.5707"/>
-      <geometry>
-        <cylinder radius="0.0325" length="0.03"/>
-      </geometry>
-    </visual>
+    <visual name="front_left_wheel_visual">
+      <origin xyz="0 0 0" rpy="0 1.5707 1.5707"/>
+      <geometry>
+        <cylinder radius="0.0325" length="0.03"/>
+      </geometry>
+    </visual>
+    <collision name="collision_front_left_wheel">
+      <origin xyz="0 0 0" rpy="0 1.5707 1.5707"/>
+      <geometry>
+        <cylinder radius="0.0325" length="0.03"/>
+      </geometry>
+    </collision>
   </link>
   <link name="front_right_wheel">
-    <collision name="collision">
-      <origin xyz="0 0 0" rpy="0 1.5707 1.5707"/>
-      <geometry>
-        <cylinder radius="0.0325" length="0.03"/>
-      </geometry>
-    </collision>
-    <visual name="right_wheel_visual">
+    <visual name="front_right_wheel_visual">
       <origin xyz="0 0 0.0" rpy="0 1.5707 1.5707"/>
       <geometry>
@@ -57,6 +48,12 @@
       </geometry>
     </visual>
-  </link>
-  <joint type="continuous" name="front_left_wheel_hinge">
+    <collision name="collision_front_right_wheel">
+      <origin xyz="0 0 0" rpy="0 1.5707 1.5707"/>
+      <geometry>
+        <cylinder radius="0.0325" length="0.03"/>
+      </geometry>
+    </collision>
+  </link>
+  <joint name="front_left_wheel_hinge" type="continuous">
     <origin xyz="0.1035 0.09 0.019" rpy="0 0 0"/>
     <child link="front_left_wheel"/>
@@ -66,5 +63,5 @@
     <joint_properties damping="1.0" friction="1.0"/>
   </joint>
-  <joint type="continuous" name="front_right_wheel_hinge">
+  <joint name="front_right_wheel_hinge" type="continuous">
     <origin xyz="0.1035 -0.09 0.019" rpy="0 0 0"/>
     <child link="front_right_wheel"/>
@@ -75,32 +72,32 @@
   </joint>
   <link name="rear_left_wheel">
-    <collision name="collision">
-      <origin xyz="0 0 0" rpy="0 1.5707 1.5707"/>
-      <geometry>
-        <cylinder radius="0.0325" length="0.03"/>
-      </geometry>
-    </collision>
-    <visual name="left_wheel_visual">
-      <origin xyz="0 0 0" rpy="0 1.5707 1.5707"/>
-      <geometry>
-        <cylinder radius="0.0325" length="0.03"/>
-      </geometry>
-    </visual>
+    <visual name="rear_left_wheel_visual">
+      <origin xyz="0 0 0" rpy="0 1.5707 1.5707"/>
+      <geometry>
+        <cylinder radius="0.0325" length="0.03"/>
+      </geometry>
+    </visual>
+    <collision name="collision_rear_left_wheel">
+      <origin xyz="0 0 0" rpy="0 1.5707 1.5707"/>
+      <geometry>
+        <cylinder radius="0.0325" length="0.03"/>
+      </geometry>
+    </collision>
   </link>
   <link name="rear_right_wheel">
-    <collision name="collision">
-      <origin xyz="0 0 0" rpy="0 1.5707 1.5707"/>
-      <geometry>
-        <cylinder radius="0.0325" length="0.03"/>
-      </geometry>
-    </collision>
-    <visual name="right_wheel_visual">
-      <origin xyz="0 0 0" rpy="0 1.5707 1.5707"/>
-      <geometry>
-        <cylinder radius="0.0325" length="0.03"/>
-      </geometry>
-    </visual>
-  </link>
-  <joint type="continuous" name="rear_left_wheel_hinge">
+    <visual name="rear_right_wheel_visual">
+      <origin xyz="0 0 0" rpy="0 1.5707 1.5707"/>
+      <geometry>
+        <cylinder radius="0.0325" length="0.03"/>
+      </geometry>
+    </visual>
+    <collision name="collision_rear_right_wheel">
+      <origin xyz="0 0 0" rpy="0 1.5707 1.5707"/>
+      <geometry>
+        <cylinder radius="0.0325" length="0.03"/>
+      </geometry>
+    </collision>
+  </link>
+  <joint name="rear_left_wheel_hinge" type="continuous">
     <origin xyz="-0.1035 0.09 0.019" rpy="0 0 0"/>
     <child link="rear_left_wheel"/>
@@ -110,5 +107,5 @@
     <joint_properties damping="1.0" friction="1.0"/>
   </joint>
-  <joint type="continuous" name="rear_right_wheel_hinge">
+  <joint name="rear_right_wheel_hinge" type="continuous">
     <origin xyz="-0.1035 -0.09 0.019" rpy="0 0 0"/>
     <child link="rear_right_wheel"/>
@@ -119,17 +116,17 @@
   </joint>
   <link name="camera">
-    <collision>
+    <visual name="camera_visual">
       <origin xyz="0 0 0" rpy="0 0 0"/>
       <geometry>
         <cylinder radius="0.005" length="0.005"/>
       </geometry>
-    </collision>
-    <visual>
+      <material name="black"/>
+    </visual>
+    <collision name="collision_camera">
       <origin xyz="0 0 0" rpy="0 0 0"/>
       <geometry>
         <cylinder radius="0.005" length="0.005"/>
       </geometry>
-      <material name="black"/>
-    </visual>
+    </collision>
   </link>
   <joint name="camera_joint" type="fixed">
@@ -139,19 +136,19 @@
   </joint>
   <link name="laser">
-    <collision>
+    <visual name="laser_visual">
       <origin xyz="0 0 0" rpy="0 0 0"/>
       <geometry>
         <cylinder radius="0.03" length="0.017"/>
       </geometry>
-    </collision>
-    <visual>
+      <material name="green_black"/>
+    </visual>
+    <collision name="collision_laser">
       <origin xyz="0 0 0" rpy="0 0 0"/>
       <geometry>
         <cylinder radius="0.03" length="0.017"/>
       </geometry>
-      <material name="green_black"/>
-    </visual>
-  </link>
-  <joint name="lidar_joint" type="fixed">
+    </collision>
+  </link>
+  <joint name="laser_joint" type="fixed">
     <axis xyz="0 1 0" />
     <origin xyz=".0493 0 0.115" rpy="0 0 3.14"/>
@@ -160,4 +157,13 @@
   </joint>
   <link name="arm_base_connect">
+    <visual name="arm_base_connect_visual">
+      <origin xyz="0 0 0" rpy="1.57 0 1.57"/>
+      <geometry>
+        <mesh filename="package://aibot_description/meshes/arm_base_connect_cover.stl" scale="0.001 0.001 0.001"/>
+      </geometry>
+      <material name = "white">
+        <color rgba = "0.5 1 1 1"/>
+      </material>
+    </visual>
     <collision name='collision_arm_base_connect'>
      <origin xyz="0 0 0.011" rpy="0 0 0"/>
@@ -166,13 +172,4 @@
       </geometry>
     </collision>
-    <visual>
-      <origin xyz="0 0 0" rpy="1.57 0 1.57"/>
-      <geometry>
-        <mesh filename="package://aibot_description/meshes/arm_base_connect_cover.stl" scale="0.001 0.001 0.001"/>
-      </geometry>
-      <material name = "white">
-        <color rgba = "0.5 1 1 1"/>
-      </material>
-    </visual>
   </link>
   <joint name="arm_base_connect_joint" type="fixed">
@@ -182,4 +179,13 @@
   </joint>
   <link name="pump_support_link">
+    <visual name="pump_support_visual">
+      <origin xyz="0 0 0" rpy="1.57 0 1.57"/>
+      <geometry>
+        <mesh filename="package://aibot_description/meshes/pump_support.stl" scale="0.001 0.001 0.001"/>
+      </geometry>
+      <material name = "green_gray">
+        <color rgba = "0.2 0.8 0.6 1"/>
+      </material>
+    </visual>
     <collision name='collision_pump_support'>
      <origin xyz="0 0 0" rpy="0 0 0"/>
@@ -188,13 +194,4 @@
       </geometry>
     </collision>
-    <visual>
-      <origin xyz="0 0 0" rpy="1.57 0 1.57"/>
-      <geometry>
-        <mesh filename="package://aibot_description/meshes/pump_support.stl" scale="0.001 0.001 0.001"/>
-      </geometry>
-      <material name = "green_gray">
-        <color rgba = "0.2 0.8 0.6 1"/>
-      </material>
-    </visual>
   </link>
   <joint name="pump_support_joint" type="fixed">
@@ -204,11 +201,5 @@
   </joint>
   <link name="camera_support_link">
-    <collision name='collision_camera_support'>
-     <origin xyz="-0.031 0 0.025" rpy="0 0 0"/>
-      <geometry>
-        <box size="0.135 0.06 0.05"/>
-      </geometry>
-    </collision>
-    <visual>
+    <visual name="camera_support_visual">
       <geometry>
         <mesh filename="package://aibot_description/meshes/camera_support.stl" scale="0.001 0.001 0.001"/>
@@ -219,4 +210,10 @@
       </material>
     </visual>
+    <collision name='collision_camera_support'>
+     <origin xyz="-0.031 0 0.025" rpy="0 0 0"/>
+      <geometry>
+        <box size="0.135 0.06 0.05"/>
+      </geometry>
+    </collision>
   </link>
   <joint name="camera_support_joint" type="fixed">
@@ -226,5 +223,5 @@
   </joint>
   <link name="usb_camera_link">
-    <visual>
+    <visual name="usb_camera_visual">
       <geometry>
         <mesh filename="package://aibot_description/meshes/camera.stl" scale="0.001 0.001 0.001"/>
@@ -409,5 +406,5 @@
   </joint>
   <link name="sucker_joint">
-    <visual>
+    <visual name="sucker_visual">
       <geometry>
         <!-- <cylinder length="0.08" radius="0.0125"/> -->
@@ -429,5 +426,4 @@
     <parent link="joint6_flange"/>
     <child link="sucker_joint"/>
-    <!-- <origin xyz= "0 0.027 0.0125" rpy = "0 0 0"/> -->
     <origin xyz= "0 0.022 0" rpy = "0 0 0"/>
   </joint>

Commit message: fix wheel joint(TF)

File: urdf/aibot_car.urdf.xacro (robot description, xacro)
@@ -55,5 +55,5 @@
     </collision>
   </link>
-  <joint name="front_left_wheel_hinge" type="continuous">
+  <joint name="front_left_wheel_hinge" type="fixed">
     <origin xyz="0.1035 0.09 0.019" rpy="0 0 0"/>
     <child link="front_left_wheel"/>
@@ -63,5 +63,5 @@
     <joint_properties damping="1.0" friction="1.0"/>
   </joint>
-  <joint name="front_right_wheel_hinge" type="continuous">
+  <joint name="front_right_wheel_hinge" type="fixed">
     <origin xyz="0.1035 -0.09 0.019" rpy="0 0 0"/>
     <child link="front_right_wheel"/>
@@ -99,5 +99,5 @@
     </collision>
   </link>
-  <joint name="rear_left_wheel_hinge" type="continuous">
+  <joint name="rear_left_wheel_hinge" type="fixed">
     <origin xyz="-0.1035 0.09 0.019" rpy="0 0 0"/>
     <child link="rear_left_wheel"/>
@@ -107,5 +107,5 @@
     <joint_properties damping="1.0" friction="1.0"/>
   </joint>
-  <joint name="rear_right_wheel_hinge" type="continuous">
+  <joint name="rear_right_wheel_hinge" type="fixed">
     <origin xyz="-0.1035 -0.09 0.019" rpy="0 0 0"/>
     <child link="rear_right_wheel"/>

Commit message: Leo: add different models and update the launch files.

File: urdf/aibot_car.urdf.xacro (robot description, xacro)
@@ -6,5 +6,5 @@
       <origin xyz="0 0 0" rpy="1.57 0 0"/>
       <geometry>
-        <mesh filename="package://aibot_description/meshes/car_body.stl" scale="0.001 0.001 0.001"/>
+        <mesh filename="package://aibot_description/meshes/myagv/car_body.stl" scale="0.001 0.001 0.001"/>
       </geometry>
     </visual>
