Commit message: fix aibot_arm_urdf.xacro

File: urdf/arm/arm.urdf.xacro (robot description, xacro)
@@ -56,5 +56,5 @@
       <parent link="arm_base_link"/>
       <axis xyz="0 0 1" />
-      <limit effort="100.0" lower="0" upper="${2 * PI - 0.01}" velocity="0.70"/>
+      <limit effort="100.0" lower="${(-55) * PI / 180}" upper="${(270-55) * PI / 180}" velocity="0.70"/>
     </joint>
      <link name = "arm_first_link">
@@ -82,5 +82,5 @@
       <parent link="arm_base_rot_link"/>
       <axis xyz="0 1 0" />
-      <limit effort="100000.0" lower="0" upper="1.47" velocity="0"/>
+      <limit effort="100000.0" lower="${(-66) * PI / 180}" upper="${(180-66) * PI / 180}" velocity="0"/>
     </joint>
     <link name = "arm_second_motor_link">
@@ -134,5 +134,5 @@
       <parent link="arm_second_motor_link"/>
       <axis xyz="0 1 0" />
-      <limit effort="100000.0" lower="-${PI}" upper="1.47" velocity="0.833"/>
+      <limit effort="100000.0" lower="0" upper="1.47" velocity="0.833"/>
     </joint>
     <link name = "arm_second_link">
@@ -160,5 +160,5 @@
       <parent link="arm_first_link"/>
       <axis xyz="0 1 0" />
-      <limit effort="100000.0" lower="-${PI}" upper="1.47" velocity="0.833"/>
+      <limit effort="100000.0" lower="0" upper="2.45" velocity="0.833"/>
     </joint>
     <link name = "arm_third_link">
@@ -186,5 +186,5 @@
       <parent link="arm_second_link"/>
       <axis xyz="0 0 1" />
-      <limit effort="100000.0" lower="-${PI}" upper="1.47" velocity="0.833"/>
+      <limit effort="100000.0" lower="${(-98) * PI / 180}" upper="${(180-98) * PI / 180}" velocity="0.833"/>
     </joint>
     <link name = "arm_fourth_link">
@@ -212,5 +212,5 @@
       <parent link="arm_third_link"/>
       <axis xyz="0 1 0" />
-      <limit effort="100000.0" lower="-${PI}" upper="1.47" velocity="0.833"/>
+      <limit effort="100000.0" lower="${(-90) * PI / 180}" upper="${(180-90) * PI / 180}" velocity="0.833"/>
     </joint>
     <arm_simple_transmission name = "arm_base_link"             reduction = "1.0"/>

Commit message: add gripper

File: urdf/arm/arm.urdf.xacro (robot description, xacro)
@@ -17,5 +17,5 @@
         <origin xyz="0 0 0.96" rpy=" 0 0 0"/>
         <geometry>
-          <box size="0.24 0.23 1.92"/>
+          <box size="0.024 0.023 0.092"/>
         </geometry>
       </collision>
@@ -42,5 +42,5 @@
         <origin xyz="0 0 0.96" rpy=" 0 0 0"/>
         <geometry>
-          <box size="0.24 0.23 1.92"/>
+          <box size="0.024 0.023 0.092"/>
         </geometry>
       </collision>
@@ -68,5 +68,5 @@
         <origin xyz="0 0 0.96" rpy=" 0 0 0"/>
         <geometry>
-          <box size="0.24 0.23 1.92"/>
+          <box size="0.024 0.023 0.092"/>
         </geometry>
       </collision>
@@ -94,5 +94,5 @@
         <origin xyz="0.09331 0 -0.037679" rpy=" 0 0 0"/>
         <geometry>
-          <box size="2.089 0.296 0.130"/>
+          <box size="0.089 0.0296 0.0130"/>
         </geometry>
       </collision>
@@ -120,5 +120,5 @@
         <origin xyz="0.09331 0 -0.037679" rpy=" 0 0 0"/>
         <geometry>
-          <box size="2.089 0.296 0.130"/>
+          <box size="0.089 0.0296 0.0130"/>
         </geometry>
       </collision>
@@ -146,5 +146,5 @@
         <origin xyz="0.09331 0 -0.037679" rpy=" 0 0 0"/>
         <geometry>
-          <box size="2.089 0.296 0.130"/>
+          <box size="0.089 0.0296 0.0130"/>
         </geometry>
       </collision>
@@ -172,5 +172,5 @@
         <origin xyz="0.09331 0 -0.037679" rpy=" 0 0 0"/>
         <geometry>
-          <box size="2.089 0.296 0.130"/>
+          <box size="0.089 0.0296 0.0130"/>
         </geometry>
       </collision>
@@ -198,5 +198,5 @@
         <origin xyz="0.09331 0 -0.037679" rpy=" 0 0 0"/>
         <geometry>
-          <box size="2.089 0.296 0.130"/>
+          <box size="0.089 0.0296 0.0130"/>
         </geometry>
       </collision>
@@ -213,4 +213,82 @@
       <axis xyz="0 1 0" />
       <limit effort="100000.0" lower="${(-90) * PI / 180}" upper="${(180-90) * PI / 180}" velocity="0.833"/>
+    </joint>
+    <link name = "arm_fifth_link">
+      <visual>
+        <origin xyz = "0 0 0" rpy = "0 0 0"/>
+         <geometry>
+           <box size="0.03 0.01 0.02"/>
+        </geometry>
+      </visual>
+      <collision name='collision'>
+        <origin xyz="0.09331 0 -0.037679" rpy=" 0 0 0"/>
+        <geometry>
+          <box size="0.089 0.0296 0.0130"/>
+        </geometry>
+      </collision>
+      <inertial>
+        <mass value="6.0"/>
+        <origin xyz="0.09331 0 -0.037679" rpy=" 0 0 0"/>
+        <box_inertia m="6.0" x="2.089" y="0.296" z="0.130"/>
+      </inertial>
+    </link>
+    <joint type="revolute" name="arm_fifth_link_joint">
+      <origin xyz="-0.013 -0.013 0.034" rpy="0 0 0"/>
+      <child link="arm_fifth_link"/>
+      <parent link="arm_fourth_link"/>
+      <axis xyz="0 0 1" />
+      <limit effort="100000.0" lower="${(-90) * PI / 180}" upper="${(180-90) * PI / 180}" velocity="0.833"/>
+    </joint>
+     <link name = "arm_gripper_left_link">
+      <visual>
+        <origin xyz = "0 0 0" rpy = "0 0 0"/>
+         <geometry>
+           <box size="0.005 0.005 0.02"/>
+        </geometry>
+      </visual>
+      <collision name='collision'>
+        <origin xyz="0.09331 0 -0.037679" rpy=" 0 0 0"/>
+        <geometry>
+          <box size="0.089 0.0296 0.0130"/>
+        </geometry>
+      </collision>
+      <inertial>
+        <mass value="6.0"/>
+        <origin xyz="0.09331 0 -0.037679" rpy=" 0 0 0"/>
+        <box_inertia m="6.0" x="2.089" y="0.296" z="0.130"/>
+      </inertial>
+    </link>
+    <joint type="prismatic" name="arm_gripper_left_link_joint">
+      <origin xyz="0.01 0 0.02" rpy="0 0 0"/>
+      <child link="arm_gripper_left_link"/>
+      <parent link="arm_fifth_link"/>
+      <axis xyz="1 0 0" />
+      <limit effort="100000.0" lower="-0.005" upper="0" velocity="0.833"/>
+    </joint>
+    <link name = "arm_gripper_right_link">
+      <visual>
+        <origin xyz = "0 0 0" rpy = "0 0 0"/>
+         <geometry>
+           <box size="0.005 0.005 0.02"/>
+        </geometry>
+      </visual>
+      <collision name='collision'>
+        <origin xyz="0.09331 0 -0.037679" rpy=" 0 0 0"/>
+        <geometry>
+          <box size="0.089 0.0296 0.0130"/>
+        </geometry>
+      </collision>
+      <inertial>
+        <mass value="6.0"/>
+        <origin xyz="0.09331 0 -0.037679" rpy=" 0 0 0"/>
+        <box_inertia m="6.0" x="2.089" y="0.296" z="0.130"/>
+      </inertial>
+    </link>
+    <joint type="prismatic" name="arm_gripper_right_link_joint">
+      <origin xyz="-0.01 0 0.02" rpy="0 0 0"/>
+      <child link="arm_gripper_right_link"/>
+      <parent link="arm_fifth_link"/>
+      <axis xyz="1 0 0" />
+      <limit effort="100000.0" lower="0" upper="0.005" velocity="0.833"/>
     </joint>
     <arm_simple_transmission name = "arm_base_link"             reduction = "1.0"/>
@@ -221,4 +299,7 @@
     <arm_simple_transmission name = "arm_third_link"            reduction = "1.0"/>
     <arm_simple_transmission name = "arm_fourth_link"           reduction = "1.0"/>
+    <arm_simple_transmission name = "arm_fifth_link"            reduction = "1.0"/>
+    <arm_simple_transmission name = "arm_gripper_left_link"     reduction = "1.0"/>
+    <arm_simple_transmission name = "arm_gripper_right_link"    reduction = "1.0"/>
     <!-- <arm_gazebo>
     </arm_gazebo> -->

Commit message: fix collision attribute

File: urdf/arm/arm.urdf.xacro (robot description, xacro)
@@ -17,5 +17,5 @@
         <origin xyz="0 0 0.96" rpy=" 0 0 0"/>
         <geometry>
-          <box size="0.024 0.023 0.092"/>
+          <box size="0.0001 0.0001 0.0001"/>
         </geometry>
       </collision>
@@ -42,5 +42,5 @@
         <origin xyz="0 0 0.96" rpy=" 0 0 0"/>
         <geometry>
-          <box size="0.024 0.023 0.092"/>
+          <box size="0.0001 0.0001 0.0001"/>
         </geometry>
       </collision>
@@ -56,5 +56,5 @@
       <parent link="arm_base_link"/>
       <axis xyz="0 0 1" />
-      <limit effort="100.0" lower="${(-55) * PI / 180}" upper="${(270-55) * PI / 180}" velocity="0.70"/>
+      <limit effort="100.0" lower="${(-55) * PI / 180}" upper="${(270-55) * PI / 180}" velocity="0.070"/>
     </joint>
      <link name = "arm_first_link">
@@ -68,5 +68,5 @@
         <origin xyz="0 0 0.96" rpy=" 0 0 0"/>
         <geometry>
-          <box size="0.024 0.023 0.092"/>
+          <box size="0.0001 0.0001 0.0001"/>
         </geometry>
       </collision>
@@ -94,5 +94,5 @@
         <origin xyz="0.09331 0 -0.037679" rpy=" 0 0 0"/>
         <geometry>
-          <box size="0.089 0.0296 0.0130"/>
+          <box size="0.0001 0.0001 0.0001"/>
         </geometry>
       </collision>
@@ -108,5 +108,5 @@
       <parent link="arm_first_link"/>
       <axis xyz="0 1 0" />
-      <limit effort="100000.0" lower="0" upper="1.47" velocity="0.833"/>
+      <limit effort="100000.0" lower="0" upper="1.47" velocity="0.0833"/>
     </joint>
     <link name = "arm_second_connector_link">
@@ -120,5 +120,5 @@
         <origin xyz="0.09331 0 -0.037679" rpy=" 0 0 0"/>
         <geometry>
-          <box size="0.089 0.0296 0.0130"/>
+          <box size="0.0001 0.0001 0.0001"/>
         </geometry>
       </collision>
@@ -134,5 +134,5 @@
       <parent link="arm_second_motor_link"/>
       <axis xyz="0 1 0" />
-      <limit effort="100000.0" lower="0" upper="1.47" velocity="0.833"/>
+      <limit effort="100000.0" lower="0" upper="1.47" velocity="0.0833"/>
     </joint>
     <link name = "arm_second_link">
@@ -146,5 +146,5 @@
         <origin xyz="0.09331 0 -0.037679" rpy=" 0 0 0"/>
         <geometry>
-          <box size="0.089 0.0296 0.0130"/>
+          <box size="0.0001 0.0001 0.0001"/>
         </geometry>
       </collision>
@@ -160,5 +160,5 @@
       <parent link="arm_first_link"/>
       <axis xyz="0 1 0" />
-      <limit effort="100000.0" lower="0" upper="2.45" velocity="0.833"/>
+      <limit effort="100000.0" lower="0" upper="2.45" velocity="0.0833"/>
     </joint>
     <link name = "arm_third_link">
@@ -172,5 +172,5 @@
         <origin xyz="0.09331 0 -0.037679" rpy=" 0 0 0"/>
         <geometry>
-          <box size="0.089 0.0296 0.0130"/>
+          <box size="0.0001 0.0001 0.0001"/>
         </geometry>
       </collision>
@@ -186,5 +186,5 @@
       <parent link="arm_second_link"/>
       <axis xyz="0 0 1" />
-      <limit effort="100000.0" lower="${(-98) * PI / 180}" upper="${(180-98) * PI / 180}" velocity="0.833"/>
+      <limit effort="100000.0" lower="${(-98) * PI / 180}" upper="${(180-98) * PI / 180}" velocity="0.0833"/>
     </joint>
     <link name = "arm_fourth_link">
@@ -198,5 +198,5 @@
         <origin xyz="0.09331 0 -0.037679" rpy=" 0 0 0"/>
         <geometry>
-          <box size="0.089 0.0296 0.0130"/>
+          <box size="0.0001 0.0001 0.0001"/>
         </geometry>
       </collision>
@@ -212,5 +212,5 @@
       <parent link="arm_third_link"/>
       <axis xyz="0 1 0" />
-      <limit effort="100000.0" lower="${(-90) * PI / 180}" upper="${(180-90) * PI / 180}" velocity="0.833"/>
+      <limit effort="100000.0" lower="${(-90) * PI / 180}" upper="${(180-90) * PI / 180}" velocity="0.0833"/>
     </joint>
     <link name = "arm_fifth_link">
@@ -224,5 +224,5 @@
         <origin xyz="0.09331 0 -0.037679" rpy=" 0 0 0"/>
         <geometry>
-          <box size="0.089 0.0296 0.0130"/>
+          <box size="0.0001 0.0001 0.0001"/>
         </geometry>
       </collision>
@@ -238,5 +238,5 @@
       <parent link="arm_fourth_link"/>
       <axis xyz="0 0 1" />
-      <limit effort="100000.0" lower="${(-90) * PI / 180}" upper="${(180-90) * PI / 180}" velocity="0.833"/>
+      <limit effort="100000.0" lower="${(-90) * PI / 180}" upper="${(180-90) * PI / 180}" velocity="0.083"/>
     </joint>
      <link name = "arm_gripper_left_link">
@@ -248,13 +248,13 @@
       </visual>
       <collision name='collision'>
-        <origin xyz="0.09331 0 -0.037679" rpy=" 0 0 0"/>
-        <geometry>
-          <box size="0.089 0.0296 0.0130"/>
-        </geometry>
-      </collision>
-      <inertial>
-        <mass value="6.0"/>
-        <origin xyz="0.09331 0 -0.037679" rpy=" 0 0 0"/>
-        <box_inertia m="6.0" x="2.089" y="0.296" z="0.130"/>
+        <origin xyz="0.01 0 0.02" rpy=" 0 0 0"/>
+        <geometry>
+          <box size="0.0001 0.0001 0.0001"/>
+        </geometry>
+      </collision>
+      <inertial>
+        <mass value="6.0"/>
+        <origin xyz="0.01 0 0.02" rpy=" 0 0 0"/>
+        <box_inertia m="6.0" x="0.005" y="0.005" z="0.02"/>
       </inertial>
     </link>
@@ -264,5 +264,5 @@
       <parent link="arm_fifth_link"/>
       <axis xyz="1 0 0" />
-      <limit effort="100000.0" lower="-0.005" upper="0" velocity="0.833"/>
+      <limit effort="100000.0" lower="-0.005" upper="0" velocity="0.005"/>
     </joint>
     <link name = "arm_gripper_right_link">
@@ -274,13 +274,13 @@
       </visual>
       <collision name='collision'>
-        <origin xyz="0.09331 0 -0.037679" rpy=" 0 0 0"/>
-        <geometry>
-          <box size="0.089 0.0296 0.0130"/>
-        </geometry>
-      </collision>
-      <inertial>
-        <mass value="6.0"/>
-        <origin xyz="0.09331 0 -0.037679" rpy=" 0 0 0"/>
-        <box_inertia m="6.0" x="2.089" y="0.296" z="0.130"/>
+        <origin xyz="-0.01 0 0.02" rpy=" 0 0 0"/>
+        <geometry>
+          <box size="0.0001 0.0001 0.0001"/>
+        </geometry>
+      </collision>
+      <inertial>
+        <mass value="6.0"/>
+        <origin xyz="-0.01 0 0.02" rpy=" 0 0 0"/>
+        <box_inertia m="6.0" x="0.005" y="0.005" z="0.02"/>
       </inertial>
     </link>
@@ -290,5 +290,5 @@
       <parent link="arm_fifth_link"/>
       <axis xyz="1 0 0" />
-      <limit effort="100000.0" lower="0" upper="0.005" velocity="0.833"/>
+      <limit effort="100000.0" lower="0" upper="0.005" velocity="0.005"/>
     </joint>
     <arm_simple_transmission name = "arm_base_link"             reduction = "1.0"/>
