Commit message: [MyAGV][WIP] add temporary inertial parameter

File: urdf/chassis/myagv/chassis.urdf.xacro (robot description, xacro)
@@ -3,4 +3,11 @@
   <link name='base_link' />
   <link name='base_footprint'>
+    <inertial>
+      <origin xyz="0 0 0" rpy="0 0 0"/>
+      <mass value="5.0" />
+      <inertia
+          ixx="0.1" iyy="0.1" izz="0.2"
+          ixy="0" ixz="0.0" iyz="0.0"/>
+    </inertial>
     <visual name='base_footprint_visual'>
       <origin xyz="0 0 0" rpy="0 1.57 3.14"/>

Commit message: [MyAGV] fix the wrong relationship between base_link and base_footprint

File: urdf/chassis/myagv/chassis.urdf.xacro (robot description, xacro)
@@ -1,6 +1,6 @@
 <?xml version='1.0'?>
 <robot name="aibot" xmlns:xacro="http://ros.org/wiki/xacro">
-  <link name='base_link' />
-  <link name='base_footprint'>
+  <link name="base_footprint" />
+  <link name="base_link">
     <inertial>
       <origin xyz="0 0 0" rpy="0 0 0"/>
@@ -29,8 +29,8 @@
     </collision>
   </link>
-  <joint name="base_footprint_joint" type="fixed" >
+  <joint name="base_link_joint" type="fixed" >
     <origin xyz="0 0 0.021" rpy="0 0 0"/>
-    <child link="base_footprint"/>
-    <parent link="base_link"/>
+    <child link="base_link"/>
+    <parent link="base_footprint"/>
   </joint>
   <link name="front_left_wheel">
@@ -65,5 +65,5 @@
     <origin xyz="0.1035 0.09 0.019" rpy="0 0 0"/>
     <child link="front_left_wheel"/>
-    <parent link="base_footprint"/>
+    <parent link="base_link"/>
     <axis xyz="0 1 0" rpy="0 0 0"/>
     <limit effort="10000" velocity="1000"/>
@@ -73,5 +73,5 @@
     <origin xyz="0.1035 -0.09 0.019" rpy="0 0 0"/>
     <child link="front_right_wheel"/>
-    <parent link="base_footprint"/>
+    <parent link="base_link"/>
     <axis xyz="0 1 0" rpy="0 0 0"/>
     <limit effort="10000" velocity="1000"/>
@@ -109,5 +109,5 @@
     <origin xyz="-0.1035 0.09 0.019" rpy="0 0 0"/>
     <child link="rear_left_wheel"/>
-    <parent link="base_footprint"/>
+    <parent link="base_link"/>
     <axis xyz="0 1 0" rpy="0 0 0"/>
     <limit effort="10000" velocity="1000"/>
@@ -117,5 +117,5 @@
     <origin xyz="-0.1035 -0.09 0.019" rpy="0 0 0"/>
     <child link="rear_right_wheel"/>
-    <parent link="base_footprint"/>
+    <parent link="base_link"/>
     <axis xyz="0 1 0" rpy="0 0 0"/>
     <limit effort="10000" velocity="1000"/>
@@ -139,5 +139,5 @@
   <joint name="camera_joint" type="fixed">
     <origin xyz=".1488 0 0.0547" rpy="1.57 0 1.57"/>
-    <parent link="base_footprint"/>
+    <parent link="base_link"/>
     <child link="camera"/>
   </joint>
@@ -160,5 +160,5 @@
     <axis xyz="0 1 0" />
     <origin xyz=".0493 0 0.115" rpy="0 0 3.14"/>
-    <parent link="base_footprint"/>
+    <parent link="base_link"/>
     <child link="laser"/>
   </joint>
@@ -174,5 +174,5 @@
   <joint name="imu_joint" type="fixed">
     <origin xyz="-0.035 -0.01 0.0216" rpy="0 0 0"/>
-    <parent link="base_footprint"/>
+    <parent link="base_link"/>
     <child link="imu_link"/>
   </joint>
@@ -188,5 +188,5 @@
   <joint name="extend_back_link_joint" type="fixed">
     <origin xyz="-0.0705 0 0.084" rpy="0 0 0"/>
-    <parent link="base_footprint"/>
+    <parent link="base_link"/>
     <child link="extend_back_link"/>
   </joint>
@@ -202,5 +202,5 @@
   <joint name="extend_front_link_joint" type="fixed">
     <origin xyz="0.0695 0 0.154" rpy="0 0 0"/>
-    <parent link="base_footprint"/>
+    <parent link="base_link"/>
     <child link="extend_front_link"/>
   </joint>

Commit message: [MyAGV] remove the env variable which is unecessary

File: urdf/chassis/myagv/chassis.urdf.xacro (robot description, xacro)
@@ -13,5 +13,5 @@
       <origin xyz="0 0 0" rpy="0 1.57 3.14"/>
       <geometry>
-        <mesh filename="package://aibot_description/meshes/$(env AIBOT_BASE)/car_body.stl" scale="0.001 0.001 0.001"/>
+        <mesh filename="package://aibot_description/meshes/myagv/car_body.stl" scale="0.001 0.001 0.001"/>
       </geometry>
     </visual>
