Commit message: yetj: add aibot_mini model

File: urdf/chassis/mini/aibot_mini.urdf.xacro (robot description, xacro)
@@ -4,24 +4,18 @@
   <link name='base_footprint'>
     <visual name='base_footprint_visual'>
-      <origin xyz="0 0 0" rpy="1.57 0 0"/>
+      <origin xyz="0 0 0" rpy="0 0 1.57"/>
       <geometry>
-        <mesh filename="package://aibot_description/meshes/a1/car_body.stl" scale="0.001 0.001 0.001"/>
+        <mesh filename="package://aibot_description/meshes/mini/car_body.stl" scale="0.001 0.001 0.001"/>
       </geometry>
     </visual>
     <collision name='collision_body'>
-    <origin xyz="0 0 0.045" rpy="0 0 0"/>
+    <origin xyz="0 0 0" rpy="0 0 0"/>
       <geometry>
-        <box size="0.32 0.18 0.09"/>
-      </geometry>
-    </collision>
-    <collision name='collision_head'>
-     <origin xyz="0.045 0 0.055" rpy="0 0 0"/>
-      <geometry>
-        <box size="0.12 0.1 0.11"/>
+        <box size="0.135 0.118 0.112"/>
       </geometry>
     </collision>
   </link>
   <joint name="base_footprint_joint" type="fixed" >
-    <origin xyz="0 0 0.0135" rpy="0 0 0"/>
+    <origin xyz="0 0 0.004" rpy="0 0 0"/>
     <child link="base_footprint"/>
     <parent link="base_link"/>
@@ -31,5 +25,5 @@
       <origin xyz="0 0 0" rpy="0 1.5707 1.5707"/>
       <geometry>
-        <cylinder radius="0.0325" length="0.03"/>
+        <cylinder radius="0.025" length="0.025"/>
       </geometry>
     </visual>
@@ -37,5 +31,5 @@
       <origin xyz="0 0 0" rpy="0 1.5707 1.5707"/>
       <geometry>
-        <cylinder radius="0.0325" length="0.03"/>
+        <cylinder radius="0.025" length="0.025"/>
       </geometry>
     </collision>
@@ -45,5 +39,5 @@
       <origin xyz="0 0 0.0" rpy="0 1.5707 1.5707"/>
       <geometry>
-        <cylinder radius="0.0325" length="0.03"/>
+        <cylinder radius="0.025" length="0.025"/>
       </geometry>
     </visual>
@@ -51,10 +45,10 @@
       <origin xyz="0 0 0" rpy="0 1.5707 1.5707"/>
       <geometry>
-        <cylinder radius="0.0325" length="0.03"/>
+        <cylinder radius="0.025" length="0.025"/>
       </geometry>
     </collision>
   </link>
   <joint name="front_left_wheel_hinge" type="fixed">
-    <origin xyz="0.1035 0.09 0.019" rpy="0 0 0"/>
+    <origin xyz="0.027 0.045 0.021" rpy="0 0 0"/>
     <child link="front_left_wheel"/>
     <parent link="base_footprint"/>
@@ -64,5 +58,5 @@
   </joint>
   <joint name="front_right_wheel_hinge" type="fixed">
-    <origin xyz="0.1035 -0.09 0.019" rpy="0 0 0"/>
+    <origin xyz="0.027 -0.045 0.021" rpy="0 0 0"/>
     <child link="front_right_wheel"/>
     <parent link="base_footprint"/>
@@ -75,5 +69,5 @@
       <origin xyz="0 0 0" rpy="0 1.5707 1.5707"/>
       <geometry>
-        <cylinder radius="0.0325" length="0.03"/>
+        <cylinder radius="0.025" length="0.025"/>
       </geometry>
     </visual>
@@ -81,5 +75,5 @@
       <origin xyz="0 0 0" rpy="0 1.5707 1.5707"/>
       <geometry>
-        <cylinder radius="0.0325" length="0.03"/>
+        <cylinder radius="0.025" length="0.025"/>
       </geometry>
     </collision>
@@ -89,5 +83,5 @@
       <origin xyz="0 0 0" rpy="0 1.5707 1.5707"/>
       <geometry>
-        <cylinder radius="0.0325" length="0.03"/>
+        <cylinder radius="0.025" length="0.025"/>
       </geometry>
     </visual>
@@ -95,10 +89,10 @@
       <origin xyz="0 0 0" rpy="0 1.5707 1.5707"/>
       <geometry>
-        <cylinder radius="0.0325" length="0.03"/>
+        <cylinder radius="0.025" length="0.025"/>
       </geometry>
     </collision>
   </link>
   <joint name="rear_left_wheel_hinge" type="fixed">
-    <origin xyz="-0.1035 0.09 0.019" rpy="0 0 0"/>
+    <origin xyz="-0.027 0.045 0.021" rpy="0 0 0"/>
     <child link="rear_left_wheel"/>
     <parent link="base_footprint"/>
@@ -108,5 +102,5 @@
   </joint>
   <joint name="rear_right_wheel_hinge" type="fixed">
-    <origin xyz="-0.1035 -0.09 0.019" rpy="0 0 0"/>
+    <origin xyz="-0.027 -0.045 0.021" rpy="0 0 0"/>
     <child link="rear_right_wheel"/>
     <parent link="base_footprint"/>
@@ -131,5 +125,5 @@
   </link>
   <joint name="camera_joint" type="fixed">
-    <origin xyz=".12 0 0.0732" rpy="1.57 0 1.57"/>
+    <origin xyz="0.065 0 0.064" rpy="1.57 0 1.57"/>
     <parent link="base_footprint"/>
     <child link="camera"/>
@@ -139,5 +133,5 @@
       <origin xyz="0 0 0" rpy="0 0 0"/>
       <geometry>
-        <cylinder radius="0.03" length="0.017"/>
+        <cylinder radius="0.028" length="0.013"/>
       </geometry>
       <material name="green_black"/>
@@ -146,5 +140,5 @@
       <origin xyz="0 0 0" rpy="0 0 0"/>
       <geometry>
-        <cylinder radius="0.03" length="0.017"/>
+        <cylinder radius="0.028" length="0.013"/>
       </geometry>
     </collision>
@@ -152,5 +146,5 @@
   <joint name="laser_joint" type="fixed">
     <axis xyz="0 1 0" />
-    <origin xyz=".0493 0 0.115" rpy="0 0 1.57"/>
+    <origin xyz="0.0325 0 0.115" rpy="0 0 1.57"/>
     <parent link="base_footprint"/>
     <child link="laser"/>
@@ -166,21 +160,7 @@
   </link>
   <joint name="imu_joint" type="fixed">
-    <origin xyz="-0.035 -0.01 0.0216" rpy="0 0 1.57"/>
+    <origin xyz="-0.017 -0.01 0.09" rpy="0 0 1.57"/>
     <parent link="base_footprint"/>
     <child link="imu_link"/>
   </joint>
-  <link name="extend_back_link">
-    <visual name="extend_visual">
-      <origin xyz="0 0 0" rpy="0 0 0"/>
-      <geometry>
-        <cylinder radius="0.001" length="0.001"/>
-      </geometry>
-      <material name="green_black"/>
-    </visual>
-  </link>
-  <joint name="extend_back_link_joint" type="fixed">
-    <origin xyz="-0.0865 0 0.088" rpy="0 0 0"/>
-    <parent link="base_footprint"/>
-    <child link="extend_back_link"/>
-  </joint>
 </robot>
