Commit message: Leo: Fix AIBot Mini collision box error!

File: urdf/chassis/mini/chassis.urdf.xacro (robot description, xacro)
@@ -11,5 +11,5 @@
     </visual>
     <collision name='collision_body'>
-    <origin xyz="0 0 0" rpy="0 0 0"/>
+    <origin xyz="0 0 0.056" rpy="0 0 0"/>
       <geometry>
         <box size="0.135 0.118 0.112"/>
