Commit message: Leo: Update models with mycobot arm.

File: urdf/chassis/a1/aibot_a1.urdf.xacro (robot description, xacro)
@@ -1,4 +1,4 @@
 <?xml version='1.0'?>
-<robot name="aibot" xmlns:xacro="http://ros.org/wiki/xacro">
+<robot name="aibot_a1" xmlns:xacro="http://ros.org/wiki/xacro">
   <link name='base_link' />
   <link name='base_footprint'>
@@ -170,3 +170,17 @@
     <child link="imu_link"/>
   </joint>
+  <link name="extend_back_link">
+    <visual name="extend_visual">
+      <origin xyz="0 0 0" rpy="0 0 0"/>
+      <geometry>
+        <cylinder radius="0.001" length="0.001"/>
+      </geometry>
+      <material name="green_black"/>
+    </visual>
+  </link>
+  <joint name="extend_back_link_joint" type="fixed">
+    <origin xyz="-0.0865 0 0.088" rpy="0 0 0"/>
+    <parent link="base_footprint"/>
+    <child link="extend_back_link"/>
+  </joint>
 </robot>

File: urdf/chassis/myagv/myagv.urdf.xacro (robot description, xacro)
@@ -170,3 +170,31 @@
     <child link="imu_link"/>
   </joint>
+  <link name="extend_back_link">
+    <visual name="extend_visual">
+      <origin xyz="0 0 0" rpy="0 0 0"/>
+      <geometry>
+        <cylinder radius="0.001" length="0.001"/>
+      </geometry>
+      <material name="green_black"/>
+    </visual>
+  </link>
+  <joint name="extend_back_link_joint" type="fixed">
+    <origin xyz="-0.0705 0 0.084" rpy="0 0 0"/>
+    <parent link="base_footprint"/>
+    <child link="extend_back_link"/>
+  </joint>
+  <link name="extend_front_link">
+    <visual name="extend_visual">
+      <origin xyz="0 0 0" rpy="0 0 0"/>
+      <geometry>
+        <cylinder radius="0.001" length="0.001"/>
+      </geometry>
+      <material name="green_black"/>
+    </visual>
+  </link>
+  <joint name="extend_front_link_joint" type="fixed">
+    <origin xyz="0.0695 0 0.154" rpy="0 0 0"/>
+    <parent link="base_footprint"/>
+    <child link="extend_front_link"/>
+  </joint>
 </robot>

File: urdf/chassis/s1/aibot_s1.urdf.xacro (robot description, xacro)
@@ -10,13 +10,7 @@
     </visual>
     <collision name='collision_body'>
-    <origin xyz="0 0 0.045" rpy="0 0 0"/>
+    <origin xyz="0 0 0.0365" rpy="0 0 0"/>
       <geometry>
-        <box size="0.32 0.18 0.09"/>
-      </geometry>
-    </collision>
-    <collision name='collision_head'>
-     <origin xyz="0.045 0 0.055" rpy="0 0 0"/>
-      <geometry>
-        <box size="0.12 0.1 0.11"/>
+        <box size="0.35 0.21 0.072"/>
       </geometry>
     </collision>

Commit message: yetj: recover aibot_a1.urdf.xacro

File: urdf/chassis/a1/aibot_a1.urdf.xacro (robot description, xacro)
@@ -152,5 +152,5 @@
   <joint name="laser_joint" type="fixed">
     <axis xyz="0 1 0" />
-    <origin xyz=".0493 0 0.115" rpy="0 0 1.57"/>
+    <origin xyz=".0493 0 0.115" rpy="0 0 3.14"/>
     <parent link="base_footprint"/>
     <child link="laser"/>
@@ -166,5 +166,5 @@
   </link>
   <joint name="imu_joint" type="fixed">
-    <origin xyz="-0.035 -0.01 0.0216" rpy="0 0 1.57"/>
+    <origin xyz="-0.035 -0.01 0.0216" rpy="0 0 0"/>
     <parent link="base_footprint"/>
     <child link="imu_link"/>
